Commit message: Update ur5_barrett.xacro
the kinect is moved from the behind to the left side of the arm as the arm was occluding kinect's view

File: Robot/ur5_barrett.xacro (robot description, xacro)
@@ -13,5 +13,6 @@
 	<!-- property list -->
 	<xacro:property name="robot_stand_height" value="0.50"/>
-	<xacro:property name="kinect_stand_length" value="0.20"/>
+	<xacro:property name="kinect_stand_length" value="0.75"/>
+	<xacro:property name="kinect_stand_distance" value="0.10"/>
 	<xacro:ur5_robot prefix="" joint_limited="false"/>
 	<!-- color macros -->
@@ -47,4 +48,18 @@
 		<visual>
 		<geometry>
+		<cylinder radius="0.03" length="${kinect_stand_distance}"/>
+		</geometry>
+		<material name="orange_transparent"/>
+		</visual>
+		<collision>
+		<geometry>
+		<cylinder radius="0.03" length="${kinect_stand_distance}"/>
+		</geometry>
+		<material name="blue_transparent"/>
+		</collision>
+	</link>
+	<link name="kinect_stand">
+		<visual>
+		<geometry>
 		<cylinder radius="0.03" length="${kinect_stand_length}"/>
 		</geometry>
@@ -54,18 +69,4 @@
 		<geometry>
 		<cylinder radius="0.03" length="${kinect_stand_length}"/>
-		</geometry>
-		<material name="blue_transparent"/>
-		</collision>
-	</link>
-	<link name="kinect_stand">
-		<visual>
-		<geometry>
-		<cylinder radius="0.03" length="${robot_stand_height*2}"/>
-		</geometry>
-		<material name="orange_transparent"/>
-		</visual>
-		<collision>
-		<geometry>
-		<cylinder radius="0.03" length="${robot_stand_height*2}"/>
 		</geometry>
 		<material name="blue_transparent"/>
@@ -88,10 +89,10 @@
 		<parent link="stand"/>
 		<child link="kinect_stand_dist"/>
-		<origin xyz="${(kinect_stand_length*0.5)+0.0735} 0 0" rpy="0 1.57 0"/>
+		<origin xyz="0 ${-(kinect_stand_distance*0.5)-0.0735} 0" rpy="1.57 0 0"/>
 	</joint>
 	<joint name="kinect_stand1" type="fixed">
 		<parent link="kinect_stand_dist"/>
 		<child link="kinect_stand"/>
-		<origin xyz="${-robot_stand_height} 0 ${kinect_stand_length*0.5}" rpy="0 -1.57 0"/>
+		<origin xyz="0 ${kinect_stand_length*0.5} ${(kinect_stand_distance*0.5)+0.015}" rpy="-1.57 0 0"/>
 	</joint>
 	<joint name="stand_to_base" type="fixed">
@@ -99,5 +100,5 @@
 		<!--child link="${arm_prefix}base_link"/-->
 		<child link="base_link"/>
-		<origin xyz="0 0 ${robot_stand_height * 0.5}" rpy="0 0 3.14"/>
+		<origin xyz="0 0 ${robot_stand_height * 0.5}" rpy="0 0 1.57"/>
 	</joint>
 </robot>

Commit message: Update ur5_barrett.xacro
the base is moved by base_link and world_frame by making the parameters x,y,z and r,p,y as 0

File: Robot/ur5_barrett.xacro (robot description, xacro)
@@ -12,6 +12,6 @@
 	<xacro:include filename="$(find ur5_barrett_description)/urdf/bh282.gazebo"/>
 	<!-- property list -->
-	<xacro:property name="robot_stand_height" value="0.50"/>
-	<xacro:property name="kinect_stand_length" value="0.75"/>
+	<xacro:property name="robot_stand_height" value="0.75"/>
+	<xacro:property name="kinect_stand_length" value="1.25"/>
 	<xacro:property name="kinect_stand_distance" value="0.10"/>
 	<xacro:ur5_robot prefix="" joint_limited="false"/>
@@ -84,5 +84,5 @@
 		<parent link="world"/>
 		<child link="stand"/>
-		<origin xyz="0 0 ${robot_stand_height * 0.5}" rpy="0 0 3.14"/>
+		<origin xyz="0 0 0" rpy="0 0 0"/>
 	</joint>
 	<joint name="base_to_kinect_stand_dist" type="fixed">

Commit message: Update ur5_barrett.xacro

File: Robot/ur5_barrett.xacro (robot description, xacro)
@@ -9,9 +9,9 @@
 	<xacro:include filename="$(find ur5_barrett_description)/urdf/kinect_properties.xacro"/>
 	<xacro:include filename="$(find ur5_barrett_description)/urdf/kinect_gazebo.urdf.xacro"/>
-	<xacro:include filename="$(find ur5_barrett_description)/urdf/bh280.urdf.xacro"/>
+	<xacro:include filename="$(find ur5_barrett_description)/urdf/bh282.urdf.xacro"/>
 	<xacro:include filename="$(find ur5_barrett_description)/urdf/bh282.gazebo"/>
 	<!-- property list -->
 	<xacro:property name="robot_stand_height" value="0.75"/>
-	<xacro:property name="kinect_stand_length" value="1.25"/>
+	<xacro:property name="kinect_stand_length" value="1"/>
 	<xacro:property name="kinect_stand_distance" value="0.10"/>
 	<xacro:ur5_robot prefix="" joint_limited="false"/>

Commit message: Update ur5_barrett.xacro

File: Robot/ur5_barrett.xacro (robot description, xacro)
@@ -13,5 +13,5 @@
 	<!-- property list -->
 	<xacro:property name="robot_stand_height" value="0.75"/>
-	<xacro:property name="kinect_stand_length" value="1"/>
+	<xacro:property name="kinect_stand_length" value="0.9"/>
 	<xacro:property name="kinect_stand_distance" value="0.10"/>
 	<xacro:ur5_robot prefix="" joint_limited="false"/>
