Commit message: The spread joints are fixed for convinience

File: urdf/bh282.urdf.xacro (robot description, xacro)
@@ -136,13 +136,13 @@
 		</link>
 		<!-- joint between BH_finger_32_link and BH_finger_33_link -->
-		<joint name="${name}_j33_joint" type="revolute">
+		<joint name="${name}_j33_joint" type="fixed">
 			<parent link="${name}_finger_32_link"/>
 			<child link="${name}_finger_33_link"/>
 			<origin xyz="-0.069936 0.003 0" rpy="0 0 0" />
-			<axis xyz="0 0 -1"/>
+			<!--axis xyz="0 0 -1"/>
 			<limit effort="${joint_effort_limit}" lower="0.0" upper="0.84" velocity="${joint_velocity_limit}"/>
-			<dynamics damping="${joint_damping}" friction="${joint_friction}"/>
-		</joint>
-		<transmission name="${name}_j33_transmission">
+			<dynamics damping="${joint_damping}" friction="${joint_friction}"/-->
+		</joint>
+		<!--transmission name="${name}_j33_transmission">
 			<type>transmission_interface/SimpleTransmission</type>
 			<joint name="${name}_j33_joint">
@@ -153,5 +153,5 @@
 			  <motorTorqueConstant>1</motorTorqueConstant>
 			</actuator>
-		</transmission>
+		</transmission-->
 		<!-- finger 1 -->
 		<!-- finger 11 link -->
@@ -177,13 +177,13 @@
 		</link>
 		<!-- joint between BH_palm_link and BH_finger_11_link -->
-		<joint name="${name}_j11_joint" type="revolute">
+		<joint name="${name}_j11_joint" type="fixed">
 			<parent link="${name}_base_link"/>
 			<child link="${name}_finger_11_link"/>
 			<origin xyz="-0.025 0 0.0252" rpy="0 0 1.5708" />
-			<axis xyz="0 0 -1"/>
+			<!--axis xyz="0 0 -1"/>
 			<limit effort="${joint_effort_limit}" lower="0" upper="3.1416" velocity="${joint_velocity_limit}"/>
-			<dynamics damping="${joint_damping}" friction="${joint_friction}"/>
-		</joint>
-		<transmission name="${name}_j11_transmission">
+			<dynamics damping="${joint_damping}" friction="${joint_friction}"/-->
+		</joint>
+		<!--transmission name="${name}_j11_transmission">
 			<type>transmission_interface/SimpleTransmission</type>
 			<joint name="${name}_j11_joint">
@@ -194,5 +194,5 @@
 			  <motorTorqueConstant>1</motorTorqueConstant>
 			</actuator>
-		</transmission>
+		</transmission-->
 		<!-- finger 12 link -->
 		<link name="${name}_finger_12_link">
@@ -260,13 +260,13 @@
 		</link>
 		<!-- joint between BH_finger_12_link and BH_finger_13_link -->
-		<joint name="${name}_j13_joint" type="revolute">
+		<joint name="${name}_j13_joint" type="fixed">
 			<parent link="${name}_finger_12_link"/>
 			<child link="${name}_finger_13_link"/>
 			<origin xyz="-0.069936 0.003 0" rpy="0 0 0" />
-			<axis xyz="0 0 -1"/>
+			<!--axis xyz="0 0 -1"/>
 			<limit effort="${joint_effort_limit}" lower="0.0" upper="0.84" velocity="${joint_velocity_limit}"/>
-			<dynamics damping="${joint_damping}" friction="${joint_friction}"/>
-		</joint>
-		<transmission name="${name}_j13_transmission">
+			<dynamics damping="${joint_damping}" friction="${joint_friction}"/-->
+		</joint>
+		<!--transmission name="${name}_j13_transmission">
 			<type>transmission_interface/SimpleTransmission</type>
 			<joint name="${name}_j13_joint">
@@ -277,5 +277,5 @@
 			  <motorTorqueConstant>1</motorTorqueConstant>
 			</actuator>
-		</transmission>
+		</transmission-->
 		<!-- finger 2 -->
 		<!-- finger 21 link -->
@@ -301,13 +301,13 @@
 		</link>
 		<!-- joint between BH_palm_link and BH_finger_21_link -->
-		<joint name="${name}_j21_joint" type="revolute">
+		<joint name="${name}_j21_joint" type="fixed">
 			<parent link="${name}_base_link"/>
 			<child link="${name}_finger_21_link"/>
 			<origin xyz="0.025 0 0.0252" rpy="0 0 1.5708" />
-			<axis xyz="0 0 1"/>
+			<!--axis xyz="0 0 1"/>
 			<limit effort="${joint_effort_limit}" lower="0" upper="3.1416" velocity="${joint_velocity_limit}"/>
-			<dynamics damping="${joint_damping}" friction="${joint_friction}"/>
-		</joint>
-		<transmission name="${name}_j21_transmission">
+			<dynamics damping="${joint_damping}" friction="${joint_friction}"/-->
+		</joint>
+		<!--transmission name="${name}_j21_transmission">
 			<type>transmission_interface/SimpleTransmission</type>
 			<joint name="${name}_j21_joint">
@@ -318,5 +318,5 @@
 			  <motorTorqueConstant>1</motorTorqueConstant>
 			</actuator>
-		</transmission>
+		</transmission-->
 		<!-- finger 12 link -->
 		<link name="${name}_finger_22_link">
@@ -384,13 +384,13 @@
 		</link>
 		<!-- joint between BH_finger_22_link and BH_finger_23_link -->
-		<joint name="${name}_j23_joint" type="revolute">
+		<joint name="${name}_j23_joint" type="fixed">
 			<parent link="${name}_finger_22_link"/>
 			<child link="${name}_finger_23_link"/>
 			<origin xyz="-0.069936 0.003 0" rpy="0 0 0" />
-			<axis xyz="0 0 -1"/>
+			<!--axis xyz="0 0 -1"/>
 			<limit effort="${joint_effort_limit}" lower="0.0" upper="0.84" velocity="${joint_velocity_limit}"/>
-			<dynamics damping="${joint_damping}" friction="${joint_friction}"/>
-		</joint>
-		<transmission name="${name}_j23_transmission">
+			<dynamics damping="${joint_damping}" friction="${joint_friction}"/-->
+		</joint>
+		<!--transmission name="${name}_j23_transmission">
 			<type>transmission_interface/SimpleTransmission</type>
 			<joint name="${name}_j23_joint">
@@ -401,5 +401,5 @@
 			  <motorTorqueConstant>1</motorTorqueConstant>
 			</actuator>
-		</transmission>
+		</transmission-->
 		<xacro:bh_gazebo name="${name}"/>
 	</xacro:macro>

Commit message: Update bh282.urdf.xacro

File: urdf/bh282.urdf.xacro (robot description, xacro)
@@ -140,6 +140,6 @@
 			<child link="${name}_finger_33_link"/>
 			<origin xyz="-0.069936 0.003 0" rpy="0 0 0" />
-			<!--axis xyz="0 0 -1"/>
-			<limit effort="${joint_effort_limit}" lower="0.0" upper="0.84" velocity="${joint_velocity_limit}"/>
+			<axis xyz="0 0 -1"/>
+			<!--limit effort="${joint_effort_limit}" lower="0.0" upper="0.84" velocity="${joint_velocity_limit}"/>
 			<dynamics damping="${joint_damping}" friction="${joint_friction}"/-->
 		</joint>
@@ -177,13 +177,13 @@
 		</link>
 		<!-- joint between BH_palm_link and BH_finger_11_link -->
-		<joint name="${name}_j11_joint" type="fixed">
+		<joint name="${name}_j11_joint" type="revolute">
 			<parent link="${name}_base_link"/>
 			<child link="${name}_finger_11_link"/>
 			<origin xyz="-0.025 0 0.0252" rpy="0 0 1.5708" />
-			<!--axis xyz="0 0 -1"/>
+			<axis xyz="0 0 -1"/>
 			<limit effort="${joint_effort_limit}" lower="0" upper="3.1416" velocity="${joint_velocity_limit}"/>
-			<dynamics damping="${joint_damping}" friction="${joint_friction}"/-->
-		</joint>
-		<!--transmission name="${name}_j11_transmission">
+			<dynamics damping="${joint_damping}" friction="${joint_friction}"/>
+		</joint>
+		<transmission name="${name}_j11_transmission">
 			<type>transmission_interface/SimpleTransmission</type>
 			<joint name="${name}_j11_joint">
@@ -194,5 +194,5 @@
 			  <motorTorqueConstant>1</motorTorqueConstant>
 			</actuator>
-		</transmission-->
+		</transmission>
 		<!-- finger 12 link -->
 		<link name="${name}_finger_12_link">
@@ -264,6 +264,6 @@
 			<child link="${name}_finger_13_link"/>
 			<origin xyz="-0.069936 0.003 0" rpy="0 0 0" />
-			<!--axis xyz="0 0 -1"/>
-			<limit effort="${joint_effort_limit}" lower="0.0" upper="0.84" velocity="${joint_velocity_limit}"/>
+			<axis xyz="0 0 -1"/>
+			<!--limit effort="${joint_effort_limit}" lower="0.0" upper="0.84" velocity="${joint_velocity_limit}"/>
 			<dynamics damping="${joint_damping}" friction="${joint_friction}"/-->
 		</joint>
@@ -301,11 +301,12 @@
 		</link>
 		<!-- joint between BH_palm_link and BH_finger_21_link -->
-		<joint name="${name}_j21_joint" type="fixed">
+		<joint name="${name}_j21_joint" type="revolute">
 			<parent link="${name}_base_link"/>
 			<child link="${name}_finger_21_link"/>
 			<origin xyz="0.025 0 0.0252" rpy="0 0 1.5708" />
-			<!--axis xyz="0 0 1"/>
+			<axis xyz="0 0 1"/>
 			<limit effort="${joint_effort_limit}" lower="0" upper="3.1416" velocity="${joint_velocity_limit}"/>
-			<dynamics damping="${joint_damping}" friction="${joint_friction}"/-->
+			<!--dynamics damping="${joint_damping}" friction="${joint_friction}"/-->
+			<mimic joint="${name}_j11_joint" multiplier="1"/>
 		</joint>
 		<!--transmission name="${name}_j21_transmission">
@@ -388,6 +389,6 @@
 			<child link="${name}_finger_23_link"/>
 			<origin xyz="-0.069936 0.003 0" rpy="0 0 0" />
-			<!--axis xyz="0 0 -1"/>
-			<limit effort="${joint_effort_limit}" lower="0.0" upper="0.84" velocity="${joint_velocity_limit}"/>
+			<axis xyz="0 0 -1"/>
+			<!--limit effort="${joint_effort_limit}" lower="0.0" upper="0.84" velocity="${joint_velocity_limit}"/>
 			<dynamics damping="${joint_damping}" friction="${joint_friction}"/-->
 		</joint>
